Commit message: unilidar

File: src/mycar_description/urdf/car.urdf.xacro (robot description, xacro)
@@ -1,5 +1,6 @@
 <robot name="mycar" xmlns:xacro="http://wiki.ros.org/xacro">
-    <xacro:include filename="car_base.urdf.xacro" />   <!--arduino -->
+    <!-- <xacro:include filename="car_base.urdf.xacro" />   arduino -->
     <!-- <xacro:include filename="car_base.urdf2.xacro" />   STM32 -->
+    <xacro:include filename="car_base_unilidar.urdf.xacro" />
     <xacro:include filename="car_camera.urdf.xacro" />
     <xacro:include filename="car_laser.urdf.xacro" />

File: src/mycar_description/urdf/car_laser.urdf.xacro (robot description, xacro)
@@ -25,5 +25,5 @@
         <origin xyz="${joint_support_x} ${joint_support_y} ${joint_support_z}" rpy="0 0 0" />
     </joint>
-    <link name="laser">
+    <link name="unilidar_imu_initial">
         <visual>
             <geometry>
@@ -35,8 +35,8 @@
         </visual>
     </link>
-    <joint name="laser2support" type="fixed">
+    <joint name="unilidar_imu_initial2support" type="fixed">
         <parent link="support" />
-        <child link="laser"/>
-        <origin xyz="${joint_laser_x} ${joint_laser_y} ${joint_laser_z}" rpy="0 0 3.1415926" />
+        <child link="unilidar_imu_initial"/>
+        <origin xyz="${joint_laser_x} ${joint_laser_y} ${joint_laser_z}" rpy="0 0 0" />
     </joint>
 </robot>
